File: pcb/motor-module/motor-module.kicad_sch (KiCad schematic)
At the start: 3 parts

Commit message: update pcb
Parts:
- added J2: Screw_Terminal_01x02, TerminalBlock_Phoenix:TerminalBlock_Phoenix_MKDS-1,5-2-5.08_1x02_P5.08mm_Horizontal, symbol Connector:Screw_Terminal_01x02
- added K1: AZ822-2C-5DSE Signal-Relais, 5 V DC, 2 A, 2 CO, Relay_THT:Relay_DPDT_Finder_30.22, symbol Relay:FINDER-30.22
- added Q1: 2N 2222A SMD Bipolartransistor, NPN, 40V, 0,8A, 0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, Package_TO_SOT_SMD:SOT-23, symbol Transistor_BJT:BC850
- added R1, R2: 1k, Resistor_SMD:R_0805_2012Metric, symbol Device:R
- D1: renamed from D?; value D -> GS1A Gleichrichterdiode, 50 V, 1 A, DO-214AC/SMA; footprint (none) -> Diode_SMD:D_SMA
- gave numbers to parts that had none: 1
Connections:
- net CMD: now reaches J1.4 (D3)
- net CMD: now also R1.2, R2.2
- net +5V: now reaches D1.1 (K)
- net +5V: now also J1.2 (+5V), K1.A1
- net sw-: now reaches D1.2 (A)
- net sw-: now also K1.A2, Q1.3 (C)
- net +12V: now reaches J1.1 (+12V)
- net +12V: now also K1.11
- net GND: now reaches J1.3 (GND)
- net GND: now also J2.1 (Pin_1), Q1.2 (E)
- new net CMD2: Q1.1 (B), R1.1, R2.1
- new net mot: J2.2 (Pin_2), K1.14
- no-connect marks 0 -> 11
Other:
- moved on the sheet: D1, J1A, J1B

Commit message: pcb update
Parts:
- removed J1: Connector_male, CAN_ATmega:Connector_male, symbol CAN_ATmega:Connector_male
- removed J2: Screw_Terminal_01x02, TerminalBlock_Phoenix:TerminalBlock_Phoenix_MKDS-1,5-2-5.08_1x02_P5.08mm_Horizontal, symbol Connector:Screw_Terminal_01x02
- added J1: Connector_male_4x8, CAN_ATmega:Connector_male_4x8, symbol CAN_ATmega:Connector_male_4x8
- added J2: Screw_Terminal_01x03, Connector_Wago:Wago_734-163_1x03_P3.50mm_Horizontal, symbol Connector:Screw_Terminal_01x03
- renumbered R1 to R1_1, R2 to R1_2
Connections:
- net +12V: now also J1.1 (+12V)
- net +5V: now also J1.2 (+5V)
- net CMD: now also J1.5 (D3)
- net GND: now also J1.4 (GND), J2.3 (Pin_3)
- net mot: now also J2.1 (Pin_1)
- no-connect marks 11 -> 13
Other:
- note added: "ATMega"
- note added: "Front Terminal"
- note added: "Power Input"
- note added: "Relay"
- moved on the sheet: D1, K1, Q1, R1_1, R1_2
