File: pcb/temp-module/temp-module.kicad_pcb (KiCad board)
At the start: 2 copper layers, 37 x 27 mm, 20 parts, among them J1 Connector_male, J2 Screw_Terminal_01x03, U1 MCP6002-xP

Commit message: new temp module
Parts:
- removed R1_1: 1.3k, Resistor_SMD:R_0805_2012Metric
- removed R1_2: 2k, Resistor_SMD:R_0805_2012Metric
- removed R1_3: 10k, Resistor_SMD:R_0805_2012Metric
- added R1: 10k, Resistor_SMD:R_0805_2012Metric, F.Cu at (151.8, 95.6)
- R2_1: value 330 -> 20.5k
- R2_2: value 1.3k -> 20.5k
- R2_3: value 110k -> 10k
- R3: value 20k -> 20.5k
- R4_1: value 2k -> 3k
- R4_2: value 2.4k -> 3k
- R4_3: value 20k -> 1k
- R5: value 1k -> 3k
- moved C3 12.3 mm to (148.3, 93.1)
- moved C2 6.35 mm to (148.3, 96.0)
- moved R3 4.19 mm to (165.6, 91.8)
- moved C4 3.54 mm to (166.2, 99.9), turned to 90 degrees
- moved R4_3 0.62 mm to (147.3, 108.0)
- moved R4_2 0.62 mm to (146.3, 110.7)
- moved R4_1 0.62 mm to (145.3, 108.0)
- moved R5 0.28 mm to (169.2, 109.1)
- moved J2 0.20 mm to (155.2, 108.4)
Connections:
- C4 pad 1: GND -> S1
- C4 pad 2: SREG -> GND
Routing:
- net GND: track 16.4 -> 6.70 mm, vias 4 -> 0
- net /vk_in: track 42.8 -> 35.4 mm
- net +5V: track 66.4 -> 60.0 mm
- net S1: track 11.9 -> 16.8 mm
- net /R_1_2_3: track 1.92 -> 0.00 mm
- net /R_1_1_2: track 1.92 -> 0.00 mm
- net /fb: track 13.3 -> 14.6 mm
- net SREG: track 17.1 -> 15.9 mm
- net /vk_buf: track 4.89 -> 6.02 mm
- net /S2: track 18.7 -> 17.8 mm
Other:
- board text removed: "R1"

Commit message: pcb update
Parts:
- removed C3: 10uF/16V, Capacitor_SMD:C_1206_3216Metric
- C1: value 100nF -> 10uF/16V
- J1: value Connector_male -> Connector_male_4x8; footprint CAN_ATmega:Connector_male -> CAN_ATmega:Connector_male_4x8
- moved C1 3.17 mm to (148.3, 95.9)
- moved C2 3.17 mm to (148.3, 92.8), turned to 0 degrees
- moved J1 1.27 mm to (158.8, 99.1)
- moved C4 0.18 mm to (166.2, 100.1)
Connections:
- C1 pad 1: +5V -> AVCC
- C2 pad 1: GND -> AVCC
- C2 pad 2: +5V -> GND
- J1 pad 2: +5V -> unconnected-(J1-Pad2)
- J1 pad 3: GND -> AVCC
- J1 pad 4: unconnected-(J1-Pad4) -> GND
- J1 pad 8: SREG -> unconnected-(J1-Pad8)
- J1 pad 9: unconnected-(J1-Pad9) -> SREG
- R3 pad 1: +5V -> AVCC
- R5 pad 2: +5V -> AVCC
- U1 pad 8: +5V -> AVCC
Routing:
- net +5V: track 60.0 -> 0.00 mm, vias 1 -> 0
- net AVCC: track 0.00 -> 58.6 mm, vias 0 -> 1
Other:
- board text removed: "GND"
