File: pcb/can-atmega/can-atmega.kicad_pcb (KiCad board)
At the start: 2 copper layers, 37 x 48 mm, 28 parts, among them J1 Screw_Terminal_01x05, J3 Conn_02x03_Odd_Even, J4 Connector_female, U1 LM1117-5.0, U2 TJA1051T, U3 MCP2515-xSO, U4 ATmega328P-A, X1 16MHz, X2 16MHz

Commit message: updated pcb
Parts:
- added L1: 10uH, Inductor_SMD:L_0805_2012Metric, B.Cu at (167.4, 109.1)
Connections:
- U1 pad 4: +5V -> (no net)
- U4 pad 18: +5V -> /AVCC
Routing:
- net +5V: track 153.7 -> 147.0 mm, vias 3 -> 2
- net /AVCC: track 0.00 -> 5.58 mm, vias 0 -> 1
Changed lines of the file:
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@@
   (net 45 "CAN_H")
   (net 46 "unconnected-(J1-Pad1)")
+  (net 47 "/AVCC")
   (footprint "Connector_IDC:IDC-Header_2x03_P2.54mm_Vertical" (layer "F.Cu")
     (at 146.5485 84.841 180)
@@
       (net 12 "U4_D13_SCK") (pinfunction "PB5") (pintype "bidirectional"))
     (pad "18" smd rect (at 4.25 2) (size 1.6 0.55) (layers "F.Cu" "F.Paste" "F.Mask")
-      (net 1 "+5V") (pinfunction "AVCC") (pintype "power_in"))
+      (net 47 "/AVCC") (pinfunction "AVCC") (pintype "power_in"))
     (pad "19" smd rect (at 4.25 1.2) (size 1.6 0.55) (layers "F.Cu" "F.Paste" "F.Mask")
       (net 19 "unconnected-(U4-Pad19)") (pinfunction "ADC6") (pintype "input+no_connect"))
@@
     )
   )
+  (footprint "Inductor_SMD:L_0805_2012Metric" (layer "B.Cu")
+    (at 167.386 109.093)
+    (descr "Inductor SMD 0805 (2012 Metric), square (rectangular) end terminal, IPC_7351 nominal, (Body size source: IPC-SM-782 page 80, https://www.pcb-3d.com/wordpress/wp-content/uploads/ipc-sm-782a_amendment_1_and_2.pdf), generated with kicad-footprint-generator")
+    (tags "inductor")
+    (property "Sheetfile" "can-atmega.kicad_sch")
+    (property "Sheetname" "")
+    (attr smd)
+    (fp_text reference "L1" (at 0 1.27) (layer "B.SilkS")
+      (effects (font (size 0.5 0.5) (thickness 0.07)) (justify mirror))
+    )
+    (fp_text value "10uH" (at 0 -1.55) (layer "B.Fab") hide
+      (effects (font (size 1 1) (thickness 0.15)) (justify mirror))
+    )
+    (fp_text user "${REFERENCE}" (at 0 0) (layer "B.Fab")
+      (effects (font (size 0.5 0.5) (thickness 0.07)) (justify mirror))
+    )
+    (fp_line (start -0.399622 -0.56) (end 0.399622 -0.56) (layer "B.SilkS") (width 0.12))
+    (fp_line (start -0.399622 0.56) (end 0.399622 0.56) (layer "B.SilkS") (width 0.12))
+    (fp_line (start 1.75 0.85) (end 1.75 -0.85) (layer "B.CrtYd") (width 0.05))
+    (fp_line (start -1.75 -0.85) (end -1.75 0.85) (layer "B.CrtYd") (width 0.05))
+    (fp_line (start -1.75 0.85) (end 1.75 0.85) (layer "B.CrtYd") (width 0.05))
+    (fp_line (start 1.75 -0.85) (end -1.75 -0.85) (layer "B.CrtYd") (width 0.05))
+    (fp_line (start -1 0.45) (end 1 0.45) (layer "B.Fab") (width 0.1))
+    (fp_line (start 1 0.45) (end 1 -0.45) (layer "B.Fab") (width 0.1))
+    (fp_line (start 1 -0.45) (end -1 -0.45) (layer "B.Fab") (width 0.1))
+    (fp_line (start -1 -0.45) (end -1 0.45) (layer "B.Fab") (width 0.1))
+    (pad "1" smd roundrect (at -1.0625 0) (size 0.875 1.2) (layers "B.Cu" "B.Paste" "B.Mask") (roundrect_rratio 0.25)
+      (net 1 "+5V") (pinfunction "1") (pintype "input"))
+    (pad "2" smd roundrect (at 1.0625 0) (size 0.875 1.2) (layers "B.Cu" "B.Paste" "B.Mask") (roundrect_rratio 0.25)
+      (net 47 "/AVCC") (pinfunction "2") (pintype "input"))
+    (model "${KICAD6_3DMODEL_DIR}/Inductor_SMD.3dshapes/L_0805_2012Metric.wrl"
+      (offset (xyz 0 0 0))
+      (scale (xyz 1 1 1))
+      (rotate (xyz 0 0 0))
+    )
+  )
   (footprint "Capacitor_SMD:C_1206_3216Metric" (layer "B.Cu")
     (at 156.718 112.014 -90)
@@
     (pad "3" smd rect (at -3.15 -2.3) (size 2 1.5) (layers "B.Cu" "B.Paste" "B.Mask")
       (net 29 "+12V") (pinfunction "VI") (pintype "power_in"))
-    (pad "4" smd rect (at 3.15 0) (size 2 3.8) (layers "B.Cu" "B.Paste" "B.Mask")
-      (net 1 "+5V"))
+    (pad "4" smd rect (at 3.15 0) (size 2 3.8) (layers "B.Cu" "B.Paste" "B.Mask"))
     (model "${KICAD6_3DMODEL_DIR}/Package_TO_SOT_SMD.3dshapes/SOT-223.wrl"
       (offset (xyz 0 0 0))
@@
   (segment (start 169.584 92.916) (end 169.466 92.916) (width 0.25) (layer "F.Cu") (net 1))
   (segment (start 143.764 100.584) (end 142.24 99.06) (width 0.25) (layer "F.Cu") (net 1))
-  (segment (start 169.386 107.182) (end 170.886 107.182) (width 0.25) (layer "F.Cu") (net 1))
   (segment (start 169.418 113.284) (end 168.91 112.776) (width 0.25) (layer "F.Cu") (net 1))
   (segment (start 168.91 112.776) (end 162.052 112.776) (width 0.25) (layer "F.Cu") (net 1))
@@
   (segment (start 147.406396 113.75) (end 142.69 109.033604) (width 0.25) (layer "F.Cu") (net 1))
   (via (at 169.466 92.916) (size 0.8) (drill 0.4) (layers "F.Cu" "B.Cu") (free) (net 1))
-  (via (at 170.886 107.182) (size 0.8) (drill 0.4) (layers "F.Cu" "B.Cu") (free) (net 1))
   (via (at 163.068 107.442) (size 0.8) (drill 0.4) (layers "F.Cu" "B.Cu") (net 1))
   (segment (start 160.729 86.409) (end 160.934 86.614) (width 0.4) (layer "B.Cu") (net 1))
+  (segment (start 163.068 108.204) (end 163.957 109.093) (width 0.25) (layer "B.Cu") (net 1))
   (segment (start 154.891 110.539) (end 153.67 111.76) (width 0.4) (layer "B.Cu") (net 1))
   (segment (start 158.242 86.409) (end 157.177 86.409) (width 0.4) (layer "B.Cu") (net 1))
   (segment (start 160.02 110.539) (end 163.068 110.539) (width 0.25) (layer "B.Cu") (net 1))
+  (segment (start 163.068 110.539) (end 163.068 109.982) (width 0.25) (layer "B.Cu") (net 1))
   (segment (start 156.718 110.539) (end 160.02 110.539) (width 0.25) (layer "B.Cu") (net 1))
-  (segment (start 164.592 108.966) (end 163.068 107.442) (width 0.25) (layer "B.Cu") (net 1))
-  (segment (start 170.886 107.182) (end 169.102 108.966) (width 0.25) (layer "B.Cu") (net 1))
   (segment (start 157.177 86.409) (end 156.718 86.868) (width 0.4) (layer "B.Cu") (net 1))
-  (segment (start 169.102 108.966) (end 164.592 108.966) (width 0.25) (layer "B.Cu") (net 1))
   (segment (start 166.673 94.185) (end 167.942 92.916) (width 0.25) (layer "B.Cu") (net 1))
   (segment (start 146.558 99.06) (end 142.24 99.06) (width 0.4) (layer "B.Cu") (net 1))
@@
   (segment (start 156.718 92.964) (end 156.718 93.472) (width 0.4) (layer "B.Cu") (net 1))
   (segment (start 153.67 111.76) (end 147.828 111.76) (width 0.4) (layer "B.Cu") (net 1))
-  (segment (start 163.068 110.49) (end 164.592 108.966) (width 0.25) (layer "B.Cu") (net 1))
+  (segment (start 163.068 109.982) (end 163.957 109.093) (width 0.25) (layer "B.Cu") (net 1))
   (segment (start 147.828 111.76) (end 146.558 110.49) (width 0.4) (layer "B.Cu") (net 1))
   (segment (start 146.558 110.49) (end 146.558 99.06) (width 0.4) (layer "B.Cu") (net 1))
@@
   (segment (start 167.234 86.614) (end 160.934 86.614) (width 0.4) (layer "B.Cu") (net 1))
   (segment (start 156.718 110.539) (end 154.891 110.539) (width 0.4) (layer "B.Cu") (net 1))
-  (segment (start 163.068 110.539) (end 163.068 110.49) (width 0.25) (layer "B.Cu") (net 1))
+  (segment (start 163.957 109.093) (end 166.3235 109.093) (width 0.25) (layer "B.Cu") (net 1))
   (segment (start 158.242 86.409) (end 160.729 86.409) (width 0.4) (layer "B.Cu") (net 1))
   (segment (start 156.718 93.472) (end 152.908 97.282) (width 0.4) (layer "B.Cu") (net 1))
@@
   (segment (start 152.908 97.282) (end 148.336 97.282) (width 0.4) (layer "B.Cu") (net 1))
   (segment (start 156.718 86.868) (end 156.718 92.964) (width 0.4) (layer "B.Cu") (net 1))
+  (segment (start 163.068 107.442) (end 163.068 108.204) (width 0.25) (layer "B.Cu") (net 1))
   (segment (start 157.353 82.042) (end 154.432 82.042) (width 1) (layer "F.Cu") (net 2))
   (segment (start 163.082 103.982) (end 162.4 103.3) (width 0.25) (layer "F.Cu") (net 2))
@@
   (segment (start 173.065 79.466) (end 173.065 81.915) (width 0.25) (layer "F.Cu") (net 45))
   (segment (start 164.719 76.962) (end 170.561 76.962) (width 0.25) (layer "F.Cu") (net 45))
+  (segment (start 169.386 107.182) (end 170.886 107.182) (width 0.25) (layer "F.Cu") (net 47))
+  (via (at 170.886 107.182) (size 0.8) (drill 0.4) (layers "F.Cu" "B.Cu") (free) (net 47))
+  (segment (start 168.4485 109.093) (end 170.434 109.093) (width 0.25) (layer "B.Cu") (net 47))
+  (segment (start 170.434 109.093) (end 170.886 108.641) (width 0.25) (layer "B.Cu") (net 47))
+  (segment (start 170.886 108.641) (end 170.886 107.182) (width 0.25) (layer "B.Cu") (net 47))
   (zone (net 0) (net_name "") (layer "B.Cu") (hatch edge 0.508)
     (connect_pads yes (clearance 0))

Commit message: pcb update
Parts:
- added C12: 22PF, Capacitor_SMD:C_1206_3216Metric, B.Cu at (152.9, 106.0)
- C10: value 22PF -> 0.1uF
- C7: value 0.1uF -> 10uF/16V
- C8: value 10uF/16V -> 0.1uF
- J4: value Connector_female -> Connector_female_4x8; footprint CAN_ATmega:Connector_female -> CAN_ATmega:Connector_female_4x8
- L1: footprint Inductor_SMD:L_0805_2012Metric -> Inductor_SMD:L_Neosid_SMS-ME3010
- LED1: footprint LED_SMD:LED_0805_2012Metric -> led_tube_MEN_12711000:led_tube_MEN_12711000
- moved R1 23.8 mm to (145.5, 108.8), turned to 0 degrees
- moved C10 21.2 mm to (169.2, 112.9), turned to 90 degrees
- moved LED1 16.3 mm to (149.5, 106.0), turned to 90 degrees
- moved C11 11.2 mm to (159.5, 103.6)
- moved C9 9.19 mm to (165.9, 112.9), turned to 90 degrees
- moved L1 6.18 mm to (162.0, 112.1)
- moved C7 5.41 mm to (154.7, 112.9)
- moved C8 5.16 mm to (158.0, 112.9)
- moved C5 2.96 mm to (151.6, 89.7), turned to -90 degrees
- moved J4 1.27 mm to (158.8, 99.1)
- moved U4 0.78 mm to (165.1, 106.0)
- moved X2 0.73 mm to (155.4, 103.6)
- moved C1 0.46 mm to (158.6, 87.6)
- moved U1 0.46 mm to (164.5, 86.4)
- moved C2 0.46 mm to (159.6, 92.5)
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Connections:
- C10 pad 1: /U4_OSC_1 -> GND
- C10 pad 2: GND -> /AREF
- C11 pad 1: GND -> /U4_OSC_1
- C11 pad 2: /U4_OSC_2 -> GND
- C9 pad 1: +5V -> GND
- C9 pad 2: GND -> AVCC
- J4 pad 10: U4_A2 -> U4_A1
- J4 pad 11: U4_A3 -> U4_A2
- J4 pad 3: GND -> AVCC
- J4 pad 4: U4_D3 -> GND
- J4 pad 5: U4_D4 -> U4_D3
- J4 pad 6: U4_D5 -> U4_D4
- J4 pad 7: U4_D6 -> U4_D5
- J4 pad 8: U4_A0 -> U4_D6
- J4 pad 9: U4_A1 -> U4_A0
- L1 pad 2: /AVCC -> AVCC
- U1 pad 4: (no net) -> +5V
- U4 pad 18: /AVCC -> AVCC
- U4 pad 20: unconnected-(U4-Pad20) -> /AREF
Routing:
- net GND: track 92.4 -> 30.9 mm, vias 15 -> 22
- net AVCC: track 0.00 -> 59.3 mm, vias 0 -> 2
- net +5V: track 147.0 -> 105.4 mm, vias 2 -> 4
- net /AREF: track 0.00 -> 9.21 mm, vias 0 -> 1
- net /U3_OSC_1: track 13.6 -> 20.5 mm
- net /AVCC: track 5.58 -> 0.00 mm, vias 1 -> 0
- net /U3_OSC_2: track 13.1 -> 16.3 mm
- net /U2_U3_TXD: track 2.88 -> 5.83 mm
- net /LED1: track 3.23 -> 6.14 mm
- net U4_RST: track 50.9 -> 48.4 mm
- net +12V: track 32.6 -> 30.8 mm
- net /U4_OSC_2: track 10.1 -> 8.56 mm
- net CAN_L: track 17.2 -> 18.2 mm
- net U4_D13_SCK: track 49.2 -> 48.2 mm
- net U4_D11_MOSI: track 50.0 -> 49.1 mm
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- added copper zone on F.Cu, net GND

Commit message: pcb fab 2025-07-04
Parts:
- C2, C7: footprint Capacitor_SMD:C_1206_3216Metric -> Capacitor_Tantalum_SMD:CP_EIA-3216-18_Kemet-A
- LED1: footprint led_tube_MEN_12711000:led_tube_MEN_12711000 -> LED_SMD:LED_0805_2012Metric; moved to B.Cu
- R1: moved to B.Cu
- moved LED1 6.92 mm to (147.7, 112.7), turned to -90 degrees
- moved R1 6.41 mm to (150.6, 112.7), turned to -90 degrees
- moved C2 0.12 mm to (159.6, 92.6)
- moved C7 0.12 mm to (154.7, 112.8)
Routing:
- net /LED1: track 6.14 -> 2.92 mm
